Commit message: Added friction to the landing pad

File: turtlebot3_gazebo/urdf/turtlebot3_waffle_pi.urdf.xacro (robot description, xacro)
@@ -314,3 +314,8 @@
   </joint>
   <link name="camera_rgb_optical_frame"/>
+  <gazebo reference="disc">
+    <material>Gazebo/Orange</material>
+      <mu1>4.01</mu1>
+      <mu2>4.01</mu2>
+  </gazebo>
 </robot>
