Commit message: Landing pad added on the turtlebot wafflepi urdf

File: turtlebot3_gazebo/models/turtlebot3_waffle_pi/org_turtlebot3_waffle_pi.urdf.xacro (robot description, xacro)
@@ -314,8 +314,3 @@
   </joint>
   <link name="camera_rgb_optical_frame"/>
-  <gazebo reference="disc">
-    <material>Gazebo/Orange</material>
-      <mu1>100.01</mu1>
-      <mu2>100.01</mu2>
-  </gazebo>
 </robot>
